Commit message: added RVIZ remotely

File: catkin_ws/src/hebi_description/urdf/4dof_4inchlow_5inchlong_robot.xacro (robot description, xacro)
@@ -30,18 +30,18 @@
   <link name="body">
     <visual>
-      <origin xyz=".145 0.2475 -.50" rpy="0 0 0" />
+      <origin xyz=".14 0.2475 -.50" rpy="0 0 0" />
       <geometry>
-        <box size="0.4 0.32 1.0" />
+        <box size="0.3 0.32 1.0" />
       </geometry>
       <xacro:silver_material/>
     </visual>
     <collision>
-      <origin xyz=".145 0.2475 -.50" rpy="0 0 0" />
+      <origin xyz=".14 0.2475 -.50" rpy="0 0 0" />
       <geometry>
-        <box size="0.4 0.32 1.0" />
+        <box size="0.3 0.32 1.0" />
       </geometry>
     </collision>
     <inertial>
-      <origin xyz=".125 .2475 -.50" rpy="0 0 0" />
+      <origin xyz=".14 .2475 -.50" rpy="0 0 0" />
       <mass value="1.0"/>
       <inertia ixx=".112" ixy="0.0" ixz="0.0" iyy=".029" iyz="0.0" izz=".0235"/>

File: catkin_ws/src/hebi_description/urdf/4dof_4inchlow_5inchlong_robot_collisions.urdf (robot description, URDF)
Before this commit: robot arm_demo, 17 links, 16 joints
Links:
- added link lower_wall, mass 1.0; collision box size=0.25 1.5 0.45; visual box size=0.25 1.5 0.45
- link body: geometry collision box size=0.4 0.32 1.0; visual box size=0.4 0.32 1.0
Joints:
- added joint lower_wall: type fixed, parent world, child lower_wall, origin xyz=-0.0606 -0.05 0.2982 rpy=0 0 0
- joint motor1/X5_9: limit lower=-0.1 upper=1.6 effort=13.0 velocity=14 -> effort=13.0 velocity=14; type revolute -> continuous
- joint motor2/X8_16: limit lower=-2.4 upper=2.4 effort=38 velocity=15 -> effort=38 velocity=15; type revolute -> continuous
- joint motor3/X5_9: limit lower=-2.5 upper=0.01 effort=13.0 velocity=14 -> effort=13.0 velocity=14; type revolute -> continuous
- joint motor4/X5_4: limit lower=-2.5 upper=0.01 effort=7.0 velocity=32 -> effort=7.0 velocity=32; type revolute -> continuous

File: catkin_ws/src/hebi_description/urdf/4dof_4inchlow_5inchlong_robot_jointlimits.urdf (robot description, URDF)
Before this commit: robot arm_demo, 17 links, 16 joints
Links:
- link body: geometry collision box size=0.4 0.32 1.0; visual box size=0.4 0.32 1.0
