Commit message: updated dof_4_lowerlonger_arm and added comments to resolved rate.

File: catkin_ws/src/hebi_description/urdf/4dof_4inchlow_5inchlong_robot.urdf (robot description, URDF)
Before this commit: robot arm_demo, 16 links, 15 joints
Links:
- link body: geometry collision box size=0.18 0.32 0.5; visual box size=0.25 0.32 1.0
- link right_arm1/INPUT_INTERFACE: mass 0.322 -> 0.32544; geometry collision cylinder length=0.1082 radius=.016; collision mesh filename=package://hebi_description/meshes/A-2038-02.stl
- link right_arm2/INPUT_INTERFACE: mass 0.36468 -> 0.36608; geometry collision cylinder length=0.2098 radius=.016; collision mesh filename=package://hebi_description/meshes/A-2038-02.stl
- link right_arm3/INPUT_INTERFACE: mass 0.35392 -> 0.35084; geometry collision cylinder length=0.1717 radius=.016; collision mesh filename=package://hebi_description/meshes/A-2038-02.stl
- link sensor/INPUT_INTERFACE: mass 0.37436 -> 0.37368; geometry collision cylinder length=0.2288 radius=.016; collision mesh filename=package://hebi_description/meshes/A-2038-02.stl
Joints:
- joint end_joint: origin xyz=0.2559 0 0.02 rpy=0 0 0 -> xyz=0.2542 0 0.02 rpy=0 0 0
- joint right_arm1/OUTPUT_JOINT: origin xyz=0.125 -0.0194432968708 0.0246859584714 rpy=1.3343 0 0 -> xyz=0.1336 -0.0194432968708 0.0246859584714 rpy=1.3343 0 0
- joint right_arm2/OUTPUT_JOINT: origin xyz=0.2317 -0.0165942524924 0.00883618415505 rpy=2.163 0 0 -> xyz=0.2352 -0.0165942524924 0.00883618415505 rpy=2.163 0 0
- joint right_arm3/OUTPUT_JOINT: origin xyz=0.2048 -0.0118153112202 0.00386313472914 rpy=-3.7736 0 0 -> xyz=0.1971 -0.0118153112202 0.00386313472914 rpy=-3.7736 0 0

File: catkin_ws/src/hebi_description/urdf/4dof_4inchlow_5inchlong_robot.xacro (robot description, xacro)
@@ -30,7 +30,7 @@
   <link name="body">
     <visual>
-      <origin xyz=".09 0.2475 -.25" rpy="0 0 0" />
+      <origin xyz=".09 0.2475 -.50" rpy="0 0 0" />
       <geometry>
-        <box size="0.25 0.32 .5" />
+        <box size="0.25 0.32 1.0" />
       </geometry>
       <xacro:silver_material/>
@@ -146,11 +146,11 @@
   <xacro:x5 joint="motor1" child="right_arm1" model="X5_9"/>
   <xacro:shoulder name="ms1" extension="0.4" twist="0"/>
-  <xacro:x_tube_link name="right_arm1" child="motor2" extension="0.125" twist="1.3343"/>
+  <xacro:x_tube_link name="right_arm1" child="motor2" extension="0.1336" twist="1.3343"/>
   <xacro:x5 joint="motor2" child="right_arm2" model="X5_9"/>
-  <xacro:x_tube_link name="right_arm2" child="motor3" extension="0.2317" twist="2.1630"/>
+  <xacro:x_tube_link name="right_arm2" child="motor3" extension="0.2352" twist="2.1630"/>
   <xacro:x5 joint="motor3" child="right_arm3" model="X5_9"/>
-  <xacro:x_tube_link name="right_arm3" child="motor4" extension="0.2048" twist="-3.7736" />
+  <xacro:x_tube_link name="right_arm3" child="motor4" extension="0.1971" twist="-3.7736" />
   <xacro:x5 joint="motor4" child="sensor" model="X5_4" />
-  <xacro:sensor_mac name="sensor" child="end_link" extension="0.2559"/>
+  <xacro:sensor_mac name="sensor" child="end_link" extension="0.2542"/>
    <!-- end link -->
   <link name="end_link/INPUT_INTERFACE">

Commit message: updated urdf model with joint limits on motor1 and motor2. resolved geometry interference with  motor1 and base link.

File: catkin_ws/src/hebi_description/urdf/4dof_4inchlow_5inchlong_robot.urdf (robot description, URDF)
Before this commit: robot arm_demo, 16 links, 15 joints
Joints:
- joint base_base: origin xyz=0 0.03 0.2984 rpy=0 0 0 -> xyz=0 0.05 0.3184 rpy=0 0 0
- joint base_s: origin xyz=0 0.03 0.2984 rpy=0 0 0 -> xyz=0 0.05 0.3184 rpy=0 0 0
- joint motor1/X5_9: limit effort=13.0 velocity=14 -> lower=-2.1 upper=1.9 effort=13.0 velocity=14; type continuous -> revolute
- joint motor2/X5_9: limit effort=13.0 velocity=14 -> lower=-2.4 upper=2.4 effort=13.0 velocity=14; type continuous -> revolute

File: catkin_ws/src/hebi_description/urdf/4dof_4inchlow_5inchlong_robot.xacro (robot description, xacro)
@@ -3,5 +3,5 @@
   <!-- *************************** XACRO MACROS *************************** -->
   <xacro:include filename="./x_library.xacro"/>
-  <xacro:include filename="./shoulder.xacro"/>
+  <xacro:include filename="./shoulder_testcopy.xacro"/>
   <xacro:include filename="./leftarm_top.xacro"/>
   <xacro:include filename="./sensor.xacro" />
@@ -121,10 +121,10 @@
     <parent link="world"/>
     <child link="motor1/INPUT_INTERFACE"/>
-    <origin xyz="0 0.03 0.2984" rpy="0 0 0"/>
+    <origin xyz="0 0.05 0.3184" rpy="0 0 0"/>
   </joint>
   <joint name="base_s" type="fixed">
     <parent link="world"/>
     <child link="ms1/INPUT_INTERFACE" />
-    <origin xyz="0 0.03 0.2984" rpy="0 0 0" />
+    <origin xyz="0 0.05 0.3184" rpy="0 0 0" />
   </joint>
   <joint name="shoulder" type="fixed">

File: catkin_ws/src/hebi_description/urdf/shoulder.xacro (robot description, xacro)
@@ -6,4 +6,5 @@
     <xacro:property name="edge_to_center" value="${.02}"/>
     <link name="${name}/INPUT_INTERFACE">
+      <!-- shifts the mount -->
       <visual>
         <origin xyz="0 0 0" rpy="${twist} 0 0" />
@@ -14,5 +15,6 @@
       </visual>
       <visual>
-        <origin xyz="${-extension/2} ${edge_to_center} 0" rpy="0 1.57075 0" />
+	<!-- shifts the bar -->
+        <origin xyz="${-extension/2} 0 ${-edge_to_center}" rpy="0 1.57075 0" />
         <geometry>
           <cylinder length="${extension-.0254}" radius=".016" />

Commit message: updated urdf to be more phat.

File: catkin_ws/src/hebi_description/urdf/4dof_4inchlow_5inchlong_robot.urdf (robot description, URDF)
Before this commit: robot arm_demo, 16 links, 15 joints
Links:
- link body: geometry collision box size=0.30 0.32 1.0; visual box size=0.30 0.32 1.0
- link head: geometry collision sphere radius=0.11; visual sphere radius=0.11
- link shoulder_len: geometry collision box size=0.12 0.8 0.8; visual box size=0.12 0.8 0.8
Joints:
- joint motor1/X5_9: limit lower=-2.1 upper=1.9 effort=13.0 velocity=14 -> effort=13.0 velocity=14; type revolute -> continuous
- joint motor2/X5_9: limit lower=-2.4 upper=2.4 effort=13.0 velocity=14 -> effort=13.0 velocity=14; type revolute -> continuous

File: catkin_ws/src/hebi_description/urdf/4dof_4inchlow_5inchlong_robot.xacro (robot description, xacro)
@@ -3,5 +3,5 @@
   <!-- *************************** XACRO MACROS *************************** -->
   <xacro:include filename="./x_library.xacro"/>
-  <xacro:include filename="./shoulder_testcopy.xacro"/>
+  <xacro:include filename="./shoulder.xacro"/>
   <xacro:include filename="./leftarm_top.xacro"/>
   <xacro:include filename="./sensor.xacro" />
@@ -10,18 +10,18 @@
   <link name="shoulder_len">
     <visual>
-      <origin xyz="0 .2475 0" rpy="0 0 0" />
+      <origin xyz="0.035 .2475 -0.08" rpy="0 0 0" />
       <geometry>
-        <box size="0.03 0.5 0.03" />
+        <box size="0.12 0.8 0.8" />
       </geometry>
       <xacro:silver_material/>
     </visual>
     <collision>
-      <origin xyz="0 -.2475 0" rpy="0 0 0" />
+      <origin xyz="0.035 -.2475 -0.08" rpy="0 0 0" />
       <geometry>
-        <box size="0.03 0.5 0.03" />
+        <box size="0.12 0.8 0.8" />
       </geometry>
     </collision>
     <inertial>
-      <origin xyz="0 .2475 0" rpy="0 0 0" />
+      <origin xyz="0.035 .2475 -0.08" rpy="0 0 0" />
       <mass value="1.0"/>
       <inertia ixx=".021" ixy="0.0" ixz="0.0" iyy=".021" iyz="0.0" izz=".00015"/>
@@ -30,18 +30,18 @@
   <link name="body">
     <visual>
-      <origin xyz=".09 0.2475 -.50" rpy="0 0 0" />
+      <origin xyz=".115 0.2475 -.50" rpy="0 0 0" />
       <geometry>
-        <box size="0.25 0.32 1.0" />
+        <box size="0.30 0.32 1.0" />
       </geometry>
       <xacro:silver_material/>
     </visual>
     <collision>
-      <origin xyz=".09 0.2475 -.25" rpy="0 0 0" />
+      <origin xyz=".115 0.2475 -.25" rpy="0 0 0" />
       <geometry>
-        <box size="0.18 0.32 0.5" />
+        <box size="0.30 0.32 1.0" />
       </geometry>
     </collision>
     <inertial>
-      <origin xyz=".09 .2475 -.25" rpy="0 0 0" />
+      <origin xyz=".115 .2475 -.25" rpy="0 0 0" />
       <mass value="1.0"/>
       <inertia ixx=".112" ixy="0.0" ixz="0.0" iyy=".029" iyz="0.0" izz=".0235"/>
@@ -52,5 +52,5 @@
       <origin xyz=".09 0.2475 .09" rpy="0 0 0" />
       <geometry>
-        <sphere radius="0.09" />
+        <sphere radius="0.11" />
       </geometry>
       <xacro:silver_material/>
@@ -59,5 +59,5 @@
       <origin xyz=".09 0.2475 .09" rpy="0 0 0" />
       <geometry>
-        <sphere radius="0.09" />
+        <sphere radius="0.11" />
       </geometry>
     </collision>
@@ -77,5 +77,5 @@
     </visual>
     <collision>
-      <origin xyz="0 -.025 -.1" rpy="0 0 0" />
+      <origin xyz="0 -.02 -.1" rpy="0 0 0" />
       <geometry>
         <box size="0.03 0.03 0.2" />
@@ -83,5 +83,5 @@
     </collision>
     <inertial>
-      <origin xyz="0 -.025 -.1" rpy="0 0 0" />
+      <origin xyz="0 -.02 -.1" rpy="0 0 0" />
       <mass value="1.0"/>
       <inertia ixx=".0034" ixy="0.0" ixz="0.0" iyy=".0034" iyz="0.0" izz=".00015"/>

Commit message: Updated camera tf frames.

File: catkin_ws/src/hebi_description/urdf/4dof_4inchlow_5inchlong_robot.urdf (robot description, URDF)
Before this commit: robot arm_demo, 16 links, 15 joints
Joints:
- joint motor1/X5_9: limit effort=13.0 velocity=14 -> lower=-2.1 upper=1.9 effort=13.0 velocity=14; type continuous -> revolute
- joint motor2/X5_9: limit effort=13.0 velocity=14 -> lower=-2.4 upper=2.4 effort=13.0 velocity=14; type continuous -> revolute
- joint motor3/X5_9: limit effort=13.0 velocity=14 -> lower=-2.5 upper=0.01 effort=13.0 velocity=14; type continuous -> revolute

Commit message: woohoo tons of random stuff

File: catkin_ws/src/hebi_description/urdf/4dof_4inchlow_5inchlong_robot.urdf (robot description, URDF)
Before this commit: robot arm_demo, 16 links, 15 joints
Joints:
- joint motor1/X5_9: limit lower=-2.1 upper=1.9 effort=13.0 velocity=14 -> lower=-0.1 upper=1.6 effort=13.0 velocity=14

Commit message: updated urdf and xacro of 4dof to incorporate 14inch low robot arm. added joint limits to motor4.

File: catkin_ws/src/hebi_description/urdf/4dof_4inchlow_5inchlong_robot.urdf (robot description, URDF)
Before this commit: robot arm_demo, 16 links, 15 joints
Joints:
- joint base_base: origin xyz=0 0.05 0.3184 rpy=0 0 0 -> xyz=0 0.05 0.2168 rpy=0 0 0
- joint base_s: origin xyz=0 0.05 0.3184 rpy=0 0 0 -> xyz=0 0.05 0.2168 rpy=0 0 0
- joint motor4/X5_4: limit effort=7.0 velocity=32 -> lower=-2.4 upper=-0.1 effort=7.0 velocity=32; type continuous -> revolute

File: catkin_ws/src/hebi_description/urdf/4dof_4inchlow_5inchlong_robot.xacro (robot description, xacro)
@@ -121,10 +121,10 @@
     <parent link="world"/>
     <child link="motor1/INPUT_INTERFACE"/>
-    <origin xyz="0 0.05 0.3184" rpy="0 0 0"/>
+    <origin xyz="0 0.05 0.2168" rpy="0 0 0"/>
   </joint>
   <joint name="base_s" type="fixed">
     <parent link="world"/>
     <child link="ms1/INPUT_INTERFACE" />
-    <origin xyz="0 0.05 0.3184" rpy="0 0 0" />
+    <origin xyz="0 0.05 0.2168" rpy="0 0 0" />
   </joint>
   <joint name="shoulder" type="fixed">

Commit message: modify vision and AM to work with new feedback and stuff

File: catkin_ws/src/hebi_description/urdf/4dof_4inchlow_5inchlong_robot.urdf (robot description, URDF)
Before this commit: robot arm_demo, 16 links, 15 joints
Joints:
- joint motor4/X5_4: limit lower=-2.4 upper=-0.1 effort=7.0 velocity=32 -> lower=-2.4 upper=0.01 effort=7.0 velocity=32

Commit message: functional push out and push up use case.

File: catkin_ws/src/hebi_description/urdf/4dof_4inchlow_5inchlong_robot.urdf (robot description, URDF)
Before this commit: robot arm_demo, 16 links, 15 joints
Joints:
- joint motor4/X5_4: limit lower=-2.4 upper=0.01 effort=7.0 velocity=32 -> lower=-2.5 upper=0.01 effort=7.0 velocity=32

Commit message: updated URDF with more safety space and included ground-level collision object.

File: catkin_ws/src/hebi_description/urdf/4dof_4inchlow_5inchlong_robot.urdf (robot description, URDF)
Before this commit: robot arm_demo, 16 links, 15 joints
Links:
- added link lower_body, mass 1.0; collision box size=1.25 1.5 0.25; visual box size=1.25 1.5 0.25
- link body: geometry collision box size=0.4 0.32 1.0; visual box size=0.4 0.32 1.0
- link head: geometry collision sphere radius=0.18; visual sphere radius=0.18
- link motor2/INPUT_INTERFACE: mass 0.322 -> 0.33; geometry collision mesh filename=package://hebi_description/meshes/X8.stl scale=0.001 0.001 0.001; visual mesh filename=package://hebi_description/meshes/X8.stl scale=0.001 0.001 0.001
- link ms1/INPUT_INTERFACE: geometry collision cylinder length=0.3746 radius=.016; collision mesh filename=package://hebi_description/meshes/A-2039-02.stl
Joints:
- removed joint motor2/X5_9
- added joint lower_body: type fixed, parent world, child lower_body, origin xyz=-0.0606 -0.05 0.2982 rpy=0 0 0
- added joint motor2/X8_16: type revolute, parent motor2/INPUT_INTERFACE, child right_arm2/INPUT_INTERFACE, origin xyz=0 0 0.045 rpy=0 0 0, axis 0 0 1, limit lower=-2.4 upper=2.4 effort=38 velocity=15
- joint base_base: origin xyz=0 0.05 0.2168 rpy=0 0 0 -> xyz=0.2794 0 0 rpy=0 0 0
- joint base_s: origin xyz=0 0.05 0.2168 rpy=0 0 0 -> xyz=0.2794 0 0 rpy=0 0 0
- joint body: origin xyz=-.34 0 0.515 rpy=0 0 0 -> xyz=-0.0606 -0.05 0.2982 rpy=0 0 0
- joint head: origin xyz=-.318 0 0.5 rpy=0 0 0 -> xyz=-0.0386 -0.05 0.2832 rpy=0 0 0
- joint left_arm: origin xyz=-.34 0.475 0.5 rpy=0 0 0 -> xyz=-0.0606 0.425 0.2832 rpy=0 0 0
- joint right_arm: origin xyz=-.34 0.03 0.5 rpy=0 0 0 -> xyz=-0.0606 -0.02 0.2832 rpy=0 0 0
- joint shoulder: origin xyz=-.34 0 0.5 rpy=0 0 0 -> xyz=-0.0606 -0.05 0.2982 rpy=0 0 0

File: catkin_ws/src/hebi_description/urdf/4dof_4inchlow_5inchlong_robot.xacro (robot description, xacro)
@@ -17,5 +17,5 @@
     </visual>
     <collision>
-      <origin xyz="0.035 -.2475 -0.08" rpy="0 0 0" />
+      <origin xyz="0.035 .2475 -0.08" rpy="0 0 0" />
       <geometry>
         <box size="0.12 0.8 0.8" />
@@ -30,18 +30,38 @@
   <link name="body">
     <visual>
-      <origin xyz=".115 0.2475 -.50" rpy="0 0 0" />
+      <origin xyz=".145 0.2475 -.50" rpy="0 0 0" />
       <geometry>
-        <box size="0.30 0.32 1.0" />
+        <box size="0.4 0.32 1.0" />
       </geometry>
       <xacro:silver_material/>
     </visual>
     <collision>
-      <origin xyz=".115 0.2475 -.25" rpy="0 0 0" />
+      <origin xyz=".145 0.2475 -.50" rpy="0 0 0" />
       <geometry>
-        <box size="0.30 0.32 1.0" />
+        <box size="0.4 0.32 1.0" />
       </geometry>
     </collision>
     <inertial>
-      <origin xyz=".115 .2475 -.25" rpy="0 0 0" />
+      <origin xyz=".125 .2475 -.50" rpy="0 0 0" />
+      <mass value="1.0"/>
+      <inertia ixx=".112" ixy="0.0" ixz="0.0" iyy=".029" iyz="0.0" izz=".0235"/>
+    </inertial>
+  </link>
+  <link name="lower_body">
+    <visual>
+      <origin xyz=".5 0.2475 -0.75" rpy="0 0 0" />
+      <geometry>
+        <box size="1.25 1.5 0.25" />
+      </geometry>
+      <xacro:silver_material/>
+    </visual>
+    <collision>
+      <origin xyz=".5 0.2475 -0.75" rpy="0 0 0" />
+      <geometry>
+        <box size="1.25 1.5 0.25" />
+      </geometry>
+    </collision>
+    <inertial>
+      <origin xyz=".5 0.2475 -0.75" rpy="0 0 0" />
       <mass value="1.0"/>
       <inertia ixx=".112" ixy="0.0" ixz="0.0" iyy=".029" iyz="0.0" izz=".0235"/>
@@ -50,18 +70,18 @@
   <link name="head">
     <visual>
-      <origin xyz=".09 0.2475 .09" rpy="0 0 0" />
+      <origin xyz=".16 0.2475 .13" rpy="0 0 0" />
       <geometry>
-        <sphere radius="0.11" />
+        <sphere radius="0.18" />
       </geometry>
       <xacro:silver_material/>
     </visual>
     <collision>
-      <origin xyz=".09 0.2475 .09" rpy="0 0 0" />
+      <origin xyz=".16 0.2475 .13" rpy="0 0 0" />
       <geometry>
-        <sphere radius="0.11" />
+        <sphere radius="0.18" />
       </geometry>
     </collision>
     <inertial>
-      <origin xyz=".09 0.2475 .09" rpy="0 0 0" />
+      <origin xyz=".09 0.2475 .13" rpy="0 0 0" />
       <mass value="1.0"/>
       <inertia ixx=".00324" ixy="0.0" ixz="0.0" iyy=".00324" iyz="0.0" izz=".00324"/>
@@ -111,41 +131,46 @@
     <parent link="world" />
     <child link="rodR" />
-    <origin xyz="-.34 0.03 0.5" rpy="0 0 0" />
+    <origin xyz="-0.0606 -0.02 0.2832" rpy="0 0 0" />
   </joint>
   <joint name="left_arm" type="fixed">
     <parent link="world" />
     <child link="rodL"/>
-    <origin xyz="-.34 0.475 0.5" rpy="0 0 0"/>
+    <origin xyz="-0.0606 0.425 0.2832" rpy="0 0 0"/>
   </joint>
   <joint name="base_base" type="fixed">
     <parent link="world"/>
     <child link="motor1/INPUT_INTERFACE"/>
-    <origin xyz="0 0.05 0.2168" rpy="0 0 0"/>
+    <origin xyz="0.2794 0 0" rpy="0 0 0"/>
   </joint>
   <joint name="base_s" type="fixed">
     <parent link="world"/>
     <child link="ms1/INPUT_INTERFACE" />
-    <origin xyz="0 0.05 0.2168" rpy="0 0 0" />
+    <origin xyz="0.2794 0 0" rpy="0 0 0" />
   </joint>
   <joint name="shoulder" type="fixed">
     <parent link="world"/>
     <child link="shoulder_len"/>
-    <origin xyz="-.34 0 0.5" rpy="0 0 0"/>
+    <origin xyz="-0.0606 -0.05 0.2982" rpy="0 0 0"/>
   </joint>
   <joint name="body" type="fixed">
     <parent link="world" />
     <child link="body" />
-    <origin xyz="-.34 0 0.515" rpy="0 0 0" />
+    <origin xyz="-0.0606 -0.05 0.2982" rpy="0 0 0" />
+  </joint>
+  <joint name="lower_body" type="fixed">
+    <parent link="world" />
+    <child link="lower_body" />
+    <origin xyz="-0.0606 -0.05 0.2982" rpy="0 0 0" />
   </joint>
   <joint name="head" type="fixed">
     <parent link="world" />
     <child link="head" />
-    <origin xyz="-.318 0 0.5" rpy="0 0 0" />
+    <origin xyz="-0.0386 -0.05 0.2832" rpy="0 0 0" />
   </joint>
   <!-- joints -->
   <xacro:x5 joint="motor1" child="right_arm1" model="X5_9"/>
-  <xacro:shoulder name="ms1" extension="0.4" twist="0"/>
+  <xacro:shoulder name="ms1" extension="0.4" twist="0.0"/>
   <xacro:x_tube_link name="right_arm1" child="motor2" extension="0.1336" twist="1.3343"/>
-  <xacro:x5 joint="motor2" child="right_arm2" model="X5_9"/>
+  <xacro:x8 joint="motor2" child="right_arm2" model="X8_16"/>
   <xacro:x_tube_link name="right_arm2" child="motor3" extension="0.2352" twist="2.1630"/>
   <xacro:x5 joint="motor3" child="right_arm3" model="X5_9"/>

File: catkin_ws/src/hebi_description/urdf/shoulder.xacro (robot description, xacro)
@@ -23,24 +23,18 @@
       </visual>
       <collision>
-        <origin xyz="0 0 0" rpy="0 ${PI/2} 0" />
+        <origin xyz="0 0 0" rpy="${twist} 0 0" />
         <geometry>
-          <mesh filename="package://hebi_description/meshes/A-2038-02.stl"/>
+          <mesh filename="package://hebi_description/meshes/A-2039-02.stl"/>
         </geometry>
       </collision>
       <collision>
-        <origin xyz="${extension/2} ${-edge_to_center} 0" rpy="0 1.57075 0" />
+        <origin xyz="${-extension/2} 0 ${-edge_to_center}" rpy="0 1.57075 0" />
         <geometry>
           <cylinder length="${extension-.0254}" radius=".016" />
         </geometry>
       </collision>
-      <collision>
-        <origin xyz="${extension} ${sin(-twist) * edge_to_center} ${edge_to_center * (1 + cos(-twist))}" rpy="${-twist} 0 0"/>
-        <geometry>
-          <mesh filename="package://hebi_description/meshes/A-2039-02.stl"/>
-        </geometry>
-      </collision>
       <!-- Approximate inertia as thin rod about x axis -->
       <inertial>
-        <origin xyz="${extension/2} 0 ${edge_to_center}" rpy="0 0 0" />
+        <origin xyz="${-extension/2} 0 ${-edge_to_center}" rpy="0 0 0" />
         <mass value="${mass}"/>
         <inertia  ixx="0.0" ixy="0.0"  ixz="0.0"  iyy="${mass * extension * extension / 12.0}"  iyz="0.0"  izz="${mass * extension * extension / 12.0}"/>

Commit message: widened URDF body to cover more of the left side of the user.

File: catkin_ws/src/hebi_description/urdf/4dof_4inchlow_5inchlong_robot.urdf (robot description, URDF)
Before this commit: robot arm_demo, 17 links, 16 joints
Links:
- link body: geometry collision box size=0.3 0.42 1.0; visual box size=0.3 0.42 1.0

File: catkin_ws/src/hebi_description/urdf/4dof_4inchlow_5inchlong_robot.xacro (robot description, xacro)
@@ -30,18 +30,18 @@
   <link name="body">
     <visual>
-      <origin xyz=".14 0.2475 -.50" rpy="0 0 0" />
+      <origin xyz=".14 0.2975 -.50" rpy="0 0 0" />
       <geometry>
-        <box size="0.3 0.32 1.0" />
+        <box size="0.3 0.42 1.0" />
       </geometry>
       <xacro:silver_material/>
     </visual>
     <collision>
-      <origin xyz=".14 0.2475 -.50" rpy="0 0 0" />
+      <origin xyz=".14 0.2975 -.50" rpy="0 0 0" />
       <geometry>
-        <box size="0.3 0.32 1.0" />
+        <box size="0.3 0.42 1.0" />
       </geometry>
     </collision>
     <inertial>
-      <origin xyz=".14 .2475 -.50" rpy="0 0 0" />
+      <origin xyz=".14 .2975 -.50" rpy="0 0 0" />
       <mass value="1.0"/>
       <inertia ixx=".112" ixy="0.0" ixz="0.0" iyy=".029" iyz="0.0" izz=".0235"/>
@@ -70,5 +70,5 @@
   <link name="head">
     <visual>
-      <origin xyz=".16 0.2475 .13" rpy="0 0 0" />
+      <origin xyz=".16 0.2875 .13" rpy="0 0 0" />
       <geometry>
         <sphere radius="0.18" />
@@ -77,5 +77,5 @@
     </visual>
     <collision>
-      <origin xyz=".16 0.2475 .13" rpy="0 0 0" />
+      <origin xyz=".16 0.2875 .13" rpy="0 0 0" />
       <geometry>
         <sphere radius="0.18" />
@@ -83,5 +83,5 @@
     </collision>
     <inertial>
-      <origin xyz=".09 0.2475 .13" rpy="0 0 0" />
+      <origin xyz=".09 0.2875 .13" rpy="0 0 0" />
       <mass value="1.0"/>
       <inertia ixx=".00324" ixy="0.0" ixz="0.0" iyy=".00324" iyz="0.0" izz=".00324"/>

File: catkin_ws/src/hebi_description/urdf/4dof_4inchlow_5inchlong_robot_jointlimits.urdf (robot description, URDF)
Before this commit: robot arm_demo, 17 links, 16 joints
Links:
- link body: geometry collision box size=0.3 0.32 1.0; visual box size=0.3 0.32 1.0
